File: instructions/untitled.sch (EAGLE design)
At the start: 27 parts, among them Q1 BC636, T1 2N3904, T2 2N3904

Commit message: updated schematic
Parts:
- removed R12: (no value), eagle-ltspice:R
- added C2, C3, C4, C5: (no value), capacitor-wima:C5/7.2
- added R13: (no value), eagle-ltspice:R
- added T3: BC547, transistor-neu-to92:BC547
Connections:
- new net +5V: R11.2, R13.1
- new net N$13: Q1.C, T3.B
- new net N$17: C5.2, R10.2, R8.1
- new net N$18: C5.1, D10.A, R11.1, T2.B
- new net SIGNAL: R13.2, SG1.-, T2.C
- net GND: now also C3.1, C4.1, D10.C, SG1.+, T2.E
- net N$12: now also C2.2, T3.C
- net N$14: now also C3.2
- net N$15: now also C2.1
- net N$16: now also C4.2, R8.2
Other:
- moved on the sheet: D10, SG1, T2
